File: KeebWithoutACase/KeebWithoutACase.kicad_pcb (KiCad board)
At the start: 2 copper layers, 133 parts, among them SW1 SW_Push_45deg, SW10 SW_Push_45deg, SW11 SW_Push_45deg, SW12 SW_Push_45deg, SW13 SW_Push_45deg, SW14 2U, SW15 1.5U, SW16 SW_Push_45deg, SW17 SW_Push_45deg, SW18 SW_Push_45deg, SW19 SW_Push_45deg, SW2 SW_Push_45deg, SW20 SW_Push_45deg, SW21 SW_Push_45deg, SW22 SW_Push_45deg, SW23 SW_Push_45deg, SW24 SW_Push_45deg, SW25 SW_Push_45deg, SW26 SW_Push_45deg, SW27 SW_Push_45deg, SW28 1.5U, SW29 1.75U, SW3 SW_Push_45deg, SW30 2.25U, SW31 SW_Push_45deg, SW32 SW_Push_45deg, SW33 SW_Push_45deg, SW34 SW_Push_45deg, SW35 SW_Push_45deg, SW36 SW_Push_45deg, SW37 SW_Push_45deg, SW38 SW_Push_45deg, SW39 SW_Push_45deg, SW4 SW_Push_45deg, SW40 SW_Push_45deg, SW41 SW_Push_45deg, SW42 SW_Push_45deg, SW43 SW_Push_45deg, SW44 SW_Push_45deg, SW45 SW_Push_45deg, SW46 SW_Push_45deg, SW47 SW_Push_45deg, SW48 SW_Push_45deg, SW49 SW_Push_45deg, SW5 SW_Push_45deg, SW50 SW_Push_45deg, SW51 SW_Push_45deg, SW52 2.75U, SW53 2.25U, SW54 1.25U, SW55 RotaryEncoder, SW56 SW_Push_45deg, SW57 1.25U, SW58 SW_Push_45deg, SW59 SW_Push_45deg, SW6 SW_Push_45deg, SW60 SW_Push_45deg, SW62 1.25U, SW63 SW_Push_45deg, SW64 SW_Push_45deg, SW65 SW_Push_45deg, SW66 SW_Push_45deg, SW67 SW_Push_45deg, SW7 SW_Push_45deg, SW8 SW_Push_45deg, SW9 SW_Push_45deg

Commit message: completed the first row of keys
Parts:
- added A1: RaspberryPi_Pico, Module:RaspberryPi_Pico_Common_Unspecified, F.Cu at (523.1, 45.1)
- moved SW39 546.5 mm to (447.0, -97.1)
- moved SW40 546.5 mm to (447.0, -82.0)
- moved SW41 546.5 mm to (447.0, -66.9)
- moved SW42 546.5 mm to (447.0, -51.8)
- moved SW43 546.5 mm to (447.0, -36.7)
- moved SW44 546.5 mm to (447.0, -21.6)
- moved SW45 546.5 mm to (447.0, -6.51)
- moved SW46 546.5 mm to (447.0, 8.57)
- moved SW47 546.5 mm to (447.0, 23.7)
- moved SW48 409.3 mm to (462.1, -97.1)
- moved SW49 409.3 mm to (462.1, -82.0)
- moved SW50 409.3 mm to (462.1, -66.9)
- moved SW51 409.3 mm to (462.1, -51.8)
- moved SW56 406.1 mm to (462.1, -21.6)
- moved SW16 384.3 mm to (401.7, -21.6)
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
Commit message: this time completed the first row with the correct keys
Parts:
- moved SW15 372.2 mm to (85.0, -113.7)
- moved SW30 361.1 mm to (182.4, -152.8)
- moved SW52 361.1 mm to (182.4, -133.0)
- moved SW53 361.1 mm to (182.4, -113.2)
- moved SW16 326.0 mm to (85.0, -98.6)
- moved SW17 326.0 mm to (85.0, -83.5)
- moved SW18 326.0 mm to (85.0, -68.4)
- moved SW19 326.0 mm to (85.0, -53.3)
- moved SW20 326.0 mm to (100.1, -174.0)
- moved SW21 326.0 mm to (100.1, -158.9)
- moved SW22 326.0 mm to (100.1, -143.8)
- moved SW23 326.0 mm to (100.1, -128.7)
- moved SW24 326.0 mm to (100.1, -113.7)
- moved SW25 326.0 mm to (100.1, -98.6)
- moved SW26 326.0 mm to (100.1, -83.5)
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Connections:
- A1 pad 9: COL 1 -> COL 2

Commit message: Row 2 complete but i forogt to commit
Parts:
- moved SW28 330.3 mm to (406.8, 69.4)
- moved SW27 314.3 mm to (382.6, 69.4)
- moved SW26 304.2 mm to (363.1, 69.5)
- moved SW25 295.8 mm to (343.5, 69.6)
- moved SW24 289.1 mm to (323.8, 69.6)
- moved SW23 284.4 mm to (304.1, 69.5)
- moved SW20 283.2 mm to (244.9, 69.4)
- moved SW22 281.8 mm to (284.2, 69.5)
- moved SW21 281.4 mm to (264.6, 69.5)
- moved SW15 191.9 mm to (142.3, 69.5)
- moved SW16 186.8 mm to (166.7, 69.5)
- moved SW19 186.4 mm to (225.3, 69.4)
- moved SW17 183.3 mm to (186.2, 69.4)
- moved SW18 183.3 mm to (205.8, 69.4)
Changed lines of the file:
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@@
 	)
 	(footprint "Button_Switch_Keyboard:SW_Cherry_MX_1.00u_PCB"
+		(locked yes)
 		(layer "F.Cu")
-		(at 84.975 -83.47)
+		(at 186.25 69.36)
 		(descr "Cherry MX keyswitch, 1.00u, PCB mount, http://cherryamericas.com/wp-content/uploads/2014/12/mx_cat.pdf")
 		(tags "Cherry MX keyswitch 1.00u PCB")
@@
 	)
 	(footprint "Button_Switch_Keyboard:SW_Cherry_MX_1.50u_PCB"
+		(locked yes)
 		(layer "F.Cu")
-		(at 84.975 -113.65)
+		(at 142.34 69.52)
 		(descr "Cherry MX keyswitch, 1.50u, PCB mount, http://cherryamericas.com/wp-content/uploads/2014/12/mx_cat.pdf")
 		(tags "Cherry MX keyswitch 1.50u PCB")
@@
 	)
 	(footprint "Button_Switch_Keyboard:SW_Cherry_MX_1.00u_PCB"
+		(locked yes)
 		(layer "F.Cu")
-		(at 100.065 -113.65)
+		(at 323.75 69.56)
 		(descr "Cherry MX keyswitch, 1.00u, PCB mount, http://cherryamericas.com/wp-content/uploads/2014/12/mx_cat.pdf")
 		(tags "Cherry MX keyswitch 1.00u PCB")
@@
 	)
 	(footprint "Button_Switch_Keyboard:SW_Cherry_MX_1.00u_PCB"
+		(locked yes)
 		(layer "F.Cu")
-		(at 100.065 -128.74)
+		(at 304.05 69.46)
 		(descr "Cherry MX keyswitch, 1.00u, PCB mount, http://cherryamericas.com/wp-content/uploads/2014/12/mx_cat.pdf")
 		(tags "Cherry MX keyswitch 1.00u PCB")
@@
 	)
 	(footprint "Button_Switch_Keyboard:SW_Cherry_MX_1.00u_PCB"
+		(locked yes)
 		(layer "F.Cu")
-		(at 100.065 -174.01)
+		(at 244.95 69.36)
 		(descr "Cherry MX keyswitch, 1.00u, PCB mount, http://cherryamericas.com/wp-content/uploads/2014/12/mx_cat.pdf")
 		(tags "Cherry MX keyswitch 1.00u PCB")
@@
 	)
 	(footprint "Button_Switch_Keyboard:SW_Cherry_MX_2.00u_PCB"
+		(locked yes)
 		(layer "F.Cu")
 		(at 401.92 49.92)
@@
 	)
 	(footprint "Button_Switch_Keyboard:SW_Cherry_MX_1.00u_PCB"
+		(locked yes)
 		(layer "F.Cu")
 		(at 157.22 49.92)
@@
 	)
 	(footprint "Button_Switch_Keyboard:SW_Cherry_MX_1.00u_PCB"
+		(locked yes)
 		(layer "F.Cu")
 		(at 372.85 49.86)
@@
 	)
 	(footprint "Button_Switch_Keyboard:SW_Cherry_MX_1.00u_PCB"
+		(locked yes)
 		(layer "F.Cu")
 		(at 235.35 49.76)
@@
 	)
 	(footprint "Button_Switch_Keyboard:SW_Cherry_MX_1.00u_PCB"
+		(locked yes)
 		(layer "F.Cu")
-		(at 84.975 -68.38)
+		(at 205.85 69.36)
 		(descr "Cherry MX keyswitch, 1.00u, PCB mount, http://cherryamericas.com/wp-content/uploads/2014/12/mx_cat.pdf")
 		(tags "Cherry MX keyswitch 1.00u PCB")
@@
 	)
 	(footprint "Button_Switch_Keyboard:SW_Cherry_MX_1.00u_PCB"
+		(locked yes)
 		(layer "F.Cu")
 		(at 353.25 49.86)
@@
 	)
 	(footprint "Button_Switch_Keyboard:SW_Cherry_MX_1.00u_PCB"
+		(locked yes)
 		(layer "F.Cu")
 		(at 314.05 49.76)
@@
 	)
 	(footprint "Button_Switch_Keyboard:SW_Cherry_MX_1.00u_PCB"
+		(locked yes)
 		(layer "F.Cu")
 		(at 215.75 49.86)
@@
 	)
 	(footprint "Button_Switch_Keyboard:SW_Cherry_MX_1.00u_PCB"
+		(locked yes)
 		(layer "F.Cu")
 		(at 137.6 49.9)
@@
 	)
 	(footprint "Button_Switch_Keyboard:SW_Cherry_MX_1.00u_PCB"
+		(locked yes)
 		(layer "F.Cu")
 		(at 274.55 49.76)
@@
 	)
 	(footprint "Button_Switch_Keyboard:SW_Cherry_MX_1.00u_PCB"
+		(locked yes)
 		(layer "F.Cu")
-		(at 100.065 -98.56)
+		(at 343.46 69.62)
 		(descr "Cherry MX keyswitch, 1.00u, PCB mount, http://cherryamericas.com/wp-content/uploads/2014/12/mx_cat.pdf")
 		(tags "Cherry MX keyswitch 1.00u PCB")
@@
 	)
 	(footprint "Button_Switch_Keyboard:SW_Cherry_MX_1.00u_PCB"
+		(locked yes)
 		(layer "F.Cu")
 		(at 294.35 49.76)
@@
 	)
 	(footprint "Button_Switch_Keyboard:SW_Cherry_MX_1.00u_PCB"
+		(locked yes)
 		(layer "F.Cu")
-		(at 84.975 -53.29)
+		(at 225.35 69.36)
 		(descr "Cherry MX keyswitch, 1.00u, PCB mount, http://cherryamericas.com/wp-content/uploads/2014/12/mx_cat.pdf")
 		(tags "Cherry MX keyswitch 1.00u PCB")
@@
 	)
 	(footprint "Button_Switch_Keyboard:SW_Cherry_MX_1.00u_PCB"
+		(locked yes)
 		(layer "F.Cu")
-		(at 84.975 -98.56)
+		(at 166.65 69.46)
 		(descr "Cherry MX keyswitch, 1.00u, PCB mount, http://cherryamericas.com/wp-content/uploads/2014/12/mx_cat.pdf")
 		(tags "Cherry MX keyswitch 1.00u PCB")
@@
 	)
 	(footprint "Button_Switch_Keyboard:SW_Cherry_MX_1.00u_PCB"
+		(locked yes)
 		(layer "F.Cu")
-		(at 100.065 -68.38)
+		(at 382.55 69.36)
 		(descr "Cherry MX keyswitch, 1.00u, PCB mount, http://cherryamericas.com/wp-content/uploads/2014/12/mx_cat.pdf")
 		(tags "Cherry MX keyswitch 1.00u PCB")
@@
 	)
 	(footprint "Button_Switch_Keyboard:SW_Cherry_MX_1.50u_PCB"
+		(locked yes)
 		(layer "F.Cu")
-		(at 100.065 -53.29)
+		(at 406.75 69.36)
 		(descr "Cherry MX keyswitch, 1.50u, PCB mount, http://cherryamericas.com/wp-content/uploads/2014/12/mx_cat.pdf")
 		(tags "Cherry MX keyswitch 1.50u PCB")
@@
 	)
 	(footprint "Button_Switch_Keyboard:SW_Cherry_MX_1.00u_PCB"
+		(locked yes)
 		(layer "F.Cu")
 		(at 196.22 49.86)
@@
 	)
 	(footprint "Button_Switch_Keyboard:SW_Cherry_MX_1.00u_PCB"
+		(locked yes)
 		(layer "F.Cu")
 		(at 176.75 49.86)
@@
 	)
 	(footprint "Button_Switch_Keyboard:SW_Cherry_MX_1.00u_PCB"
+		(locked yes)
 		(layer "F.Cu")
-		(at 100.065 -143.83)
+		(at 284.25 69.46)
 		(descr "Cherry MX keyswitch, 1.00u, PCB mount, http://cherryamericas.com/wp-content/uploads/2014/12/mx_cat.pdf")
 		(tags "Cherry MX keyswitch 1.00u PCB")
@@
 	)
 	(footprint "Button_Switch_Keyboard:SW_Cherry_MX_1.00u_PCB"
+		(locked yes)
 		(layer "F.Cu")
 		(at 333.65 49.76)
@@
 	)
 	(footprint "Button_Switch_Keyboard:SW_Cherry_MX_1.00u_PCB"
+		(locked yes)
 		(layer "F.Cu")
 		(at 254.95 49.66)
@@
 	)
 	(footprint "Button_Switch_Keyboard:SW_Cherry_MX_1.00u_PCB"
+		(locked yes)
 		(layer "F.Cu")
-		(at 100.065 -158.92)
+		(at 264.55 69.46)
 		(descr "Cherry MX keyswitch, 1.00u, PCB mount, http://cherryamericas.com/wp-content/uploads/2014/12/mx_cat.pdf")
 		(tags "Cherry MX keyswitch 1.00u PCB")
@@
 	)
 	(footprint "Button_Switch_Keyboard:SW_Cherry_MX_1.00u_PCB"
+		(locked yes)
 		(layer "F.Cu")
-		(at 100.065 -83.47)
+		(at 363.05 69.46)
 		(descr "Cherry MX keyswitch, 1.00u, PCB mount, http://cherryamericas.com/wp-content/uploads/2014/12/mx_cat.pdf")
 		(tags "Cherry MX keyswitch 1.00u PCB")
@@
 		)
 	)
+	(group ""
+		(locked yes)
+		(members "3da46f46-cf1c-489a-98e6-f911468b302e" "497997e3-6d5e-49da-a910-2333c0189895"
+			"4cf517c7-943b-4de8-8f90-04ba7088a3a0" "506364c4-b941-4a80-9a2f-4e453e524cac"
+			"62e3ee00-b798-4ad0-88a3-fa4e11150ca0" "788b491c-bb5e-4028-8c0e-b7d53d79fd01"
+			"7a0cffb1-1d89-4a7d-ac23-45a6eebbd272" "7eba087f-6283-4d93-821f-b922322d5711"
+			"81bbcee2-624b-4109-a5c4-2d8d5a0a0094" "8a2ceecb-432b-472b-bcf1-567acbcef11c"
+			"a877471d-7423-48fb-9e26-bc7fd3345d69" "b69dddbc-9b2b-4bea-808f-c26815b29701"
+			"ce6cd802-6111-4bfe-92e3-51f323804223" "e76ac1c1-c39a-44f9-88b5-9f21c8af6e78"
+		)
+	)
+	(group ""
+		(locked yes)
+		(members "27a1df57-c3fa-469b-963c-d89514c8ba91" "291d465e-5f61-4992-8adb-9aabb026c3c0"
+			"292303f4-98ba-4737-a5f2-06c9aebadcd0" "2e2b6754-0c2a-4400-afcc-3513fbfd9d6e"
+			"2fb839d3-f123-496b-82ce-349fc86f823f" "51d43e78-13da-4a40-87d4-1b0d49df645a"
+			"874009ea-9b6e-4d59-9d28-acc8f098dd08" "90c52f0c-6fac-4f49-a8dd-c836facf0909"
+			"9a7cc8ad-ffc1-4ec0-81a9-ab38b78e0da0" "9f5f9759-212f-45e2-9d43-6780ccd482b5"
+			"a17c4d75-9cb1-4170-8777-8493a7517c25" "cb72b5c5-b29e-4259-86d9-20b07935c67d"
+			"edf53278-568f-48c1-b5ad-eaa62405a4c2" "f262d881-c547-468d-9f8b-43e7fd2cfd30"
+		)
+	)

Commit message: completed arranging the third row
Parts:
- moved SW30 485.5 mm to (567.5, 142.8)
- moved SW32 485.5 mm to (500.3, 151.8)
- moved SW34 485.5 mm to (500.3, 181.9)
- moved SW36 485.5 mm to (500.3, 212.1)
- moved SW38 485.5 mm to (500.3, 242.3)
- moved SW40 485.5 mm to (515.4, 136.7)
- moved SW42 485.5 mm to (515.4, 166.8)
- moved SW44 485.5 mm to (515.4, 197.0)
- moved SW46 485.5 mm to (515.4, 227.2)
- moved SW48 485.5 mm to (530.4, 121.6)
- moved SW50 485.5 mm to (530.4, 151.8)
- moved SW52 485.5 mm to (567.5, 162.6)
- moved SW54 485.5 mm to (530.4, 181.9)
- moved SW56 485.5 mm to (530.4, 197.0)
- moved SW57 485.5 mm to (530.4, 212.1)
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
Commit message: Finished the final forkin row!!!
Parts:
- moved SW30 419.4 mm to (149.4, 108.6)
- moved SW57 399.5 mm to (139.9, 128.2)
- moved SW58 381.8 mm to (161.8, 128.2)
- moved SW59 367.5 mm to (181.2, 128.2)
- moved SW60 345.0 mm to (200.6, 128.1)
- moved SW32 322.3 mm to (180.8, 108.7)
- moved SW34 308.7 mm to (200.4, 108.7)
- moved SW36 298.6 mm to (220.1, 108.7)
- moved SW38 292.6 mm to (239.9, 108.7)
- moved SpaceBar1 263.5 mm to (271.2, 128.1)
- moved SW40 257.4 mm to (259.5, 108.7)
- moved SW42 243.2 mm to (279.2, 108.7)
- moved SW44 233.7 mm to (299.0, 108.7)
- moved SW46 229.6 mm to (318.6, 108.8)
- moved SW62 201.0 mm to (344.7, 128.2)
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Changed lines of the file:
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@@
 	)
 	(footprint "Button_Switch_Keyboard:SW_Cherry_MX_1.00u_PCB"
+		(locked yes)
 		(layer "F.Cu")
-		(at 515.35 197.03)
+		(at 299 108.7)
 		(descr "Cherry MX keyswitch, 1.00u, PCB mount, http://cherryamericas.com/wp-content/uploads/2014/12/mx_cat.pdf")
 		(tags "Cherry MX keyswitch 1.00u PCB")
@@
 	)
 	(footprint "Button_Switch_Keyboard:SW_Cherry_MX_1.00u_PCB"
+		(locked yes)
 		(layer "F.Cu")
-		(at 500.26 181.94)
+		(at 200.4 108.7)
 		(descr "Cherry MX keyswitch, 1.00u, PCB mount, http://cherryamericas.com/wp-content/uploads/2014/12/mx_cat.pdf")
 		(tags "Cherry MX keyswitch 1.00u PCB")
@@
 	)
 	(footprint "Button_Switch_Keyboard:SW_Cherry_MX_1.25u_PCB"
+		(locked yes)
 		(layer "F.Cu")
-		(at 530.44 212.12)
+		(at 139.9 128.16)
 		(descr "Cherry MX keyswitch, 1.25u, PCB mount, http://cherryamericas.com/wp-content/uploads/2014/12/mx_cat.pdf")
 		(tags "Cherry MX keyswitch 1.25u PCB")
@@
 	)
 	(footprint "Button_Switch_Keyboard:SW_Cherry_MX_1.25u_PCB"
+		(locked yes)
 		(layer "F.Cu")
-		(at 530.44 181.94)
+		(at 409.15 128.16)
 		(descr "Cherry MX keyswitch, 1.25u, PCB mount, http://cherryamericas.com/wp-content/uploads/2014/12/mx_cat.pdf")
 		(tags "Cherry MX keyswitch 1.25u PCB")
@@
 	)
 	(footprint "Button_Switch_Keyboard:SW_Cherry_MX_1.00u_PCB"
+		(locked yes)
 		(layer "F.Cu")
-		(at 500.26 151.76)
+		(at 180.8 108.7)
 		(descr "Cherry MX keyswitch, 1.00u, PCB mount, http://cherryamericas.com/wp-content/uploads/2014/12/mx_cat.pdf")
 		(tags "Cherry MX keyswitch 1.00u PCB")
@@
 	)
 	(footprint "Button_Switch_Keyboard:SW_Cherry_MX_2.25u_PCB"
+		(locked yes)
 		(layer "F.Cu")
-		(at 567.475 142.825)
+		(at 149.44 108.62)
 		(descr "Cherry MX keyswitch, 2.25u, PCB mount, http://cherryamericas.com/wp-content/uploads/2014/12/mx_cat.pdf")
 		(tags "Cherry MX keyswitch 2.25u PCB")
@@
 	)
 	(footprint "Button_Switch_Keyboard:SW_Cherry_MX_1.00u_PCB"
+		(locked yes)
 		(layer "F.Cu")
-		(at 515.35 166.85)
+		(at 279.16 108.7)
 		(descr "Cherry MX keyswitch, 1.00u, PCB mount, http://cherryamericas.com/wp-content/uploads/2014/12/mx_cat.pdf")
 		(tags "Cherry MX keyswitch 1.00u PCB")
@@
 	(footprint "Button_Switch_Keyboard:SW_Cherry_MX_1.00u_PCB"
 		(layer "F.Cu")
-		(at 530.44 197.03)
+		(at 544.29 154.32)
 		(descr "Cherry MX keyswitch, 1.00u, PCB mount, http://cherryamericas.com/wp-content/uploads/2014/12/mx_cat.pdf")
 		(tags "Cherry MX keyswitch 1.00u PCB")
@@
 	)
 	(footprint "Button_Switch_Keyboard:SW_Cherry_MX_1.00u_PCB"
+		(locked yes)
 		(layer "F.Cu")
-		(at 500.26 242.3)
+		(at 239.9 108.7)
 		(descr "Cherry MX keyswitch, 1.00u, PCB mount, http://cherryamericas.com/wp-content/uploads/2014/12/mx_cat.pdf")
 		(tags "Cherry MX keyswitch 1.00u PCB")
@@
 	)
 	(footprint "Button_Switch_Keyboard:SW_Cherry_MX_1.00u_PCB"
+		(locked yes)
 		(layer "F.Cu")
-		(at 530.44 121.58)
+		(at 338.3 108.8)
 		(descr "Cherry MX keyswitch, 1.00u, PCB mount, http://cherryamericas.com/wp-content/uploads/2014/12/mx_cat.pdf")
 		(tags "Cherry MX keyswitch 1.00u PCB")
@@
 	)
 	(footprint "Button_Switch_Keyboard:SW_Cherry_MX_1.00u_PCB"
+		(locked yes)
 		(layer "F.Cu")
-		(at 530.44 227.21)
+		(at 161.75 128.2)
 		(descr "Cherry MX keyswitch, 1.00u, PCB mount, http://cherryamericas.com/wp-content/uploads/2014/12/mx_cat.pdf")
 		(tags "Cherry MX keyswitch 1.00u PCB")
@@
 	)
 	(footprint "Button_Switch_Keyboard:SW_Cherry_MX_1.25u_PCB"
+		(locked yes)
 		(layer "F.Cu")
-		(at 545.53 136.67)
+		(at 344.66 128.17)
 		(descr "Cherry MX keyswitch, 1.25u, PCB mount, http://cherryamericas.com/wp-content/uploads/2014/12/mx_cat.pdf")
 		(tags "Cherry MX keyswitch 1.25u PCB")
@@
 	)
 	(footprint "Button_Switch_Keyboard:SW_Cherry_MX_1.00u_PCB"
+		(locked yes)
 		(layer "F.Cu")
-		(at 545.53 166.85)
+		(at 386.85 128.2)
 		(descr "Cherry MX keyswitch, 1.00u, PCB mount, http://cherryamericas.com/wp-content/uploads/2014/12/mx_cat.pdf")
 		(tags "Cherry MX keyswitch 1.00u PCB")
@@
 	)
 	(footprint "Button_Switch_Keyboard:SW_Cherry_MX_1.00u_PCB"
+		(locked yes)
 		(layer "F.Cu")
-		(at 515.35 227.21)
+		(at 318.6 108.8)
 		(descr "Cherry MX keyswitch, 1.00u, PCB mount, http://cherryamericas.com/wp-content/uploads/2014/12/mx_cat.pdf")
 		(tags "Cherry MX keyswitch 1.00u PCB")
@@
 	)
 	(footprint "Button_Switch_Keyboard:SW_Cherry_MX_1.00u_PCB"
+		(locked yes)
 		(layer "F.Cu")
-		(at 515.35 136.67)
+		(at 259.5 108.7)
 		(descr "Cherry MX keyswitch, 1.00u, PCB mount, http://cherryamericas.com/wp-content/uploads/2014/12/mx_cat.pdf")
 		(tags "Cherry MX keyswitch 1.00u PCB")
@@
 	)
 	(footprint "Button_Switch_Keyboard:SW_Cherry_MX_1.00u_PCB"
+		(locked yes)
 		(layer "F.Cu")
-		(at 545.53 151.76)
+		(at 366.95 128.1)
 		(descr "Cherry MX keyswitch, 1.00u, PCB mount, http://cherryamericas.com/wp-content/uploads/2014/12/mx_cat.pdf")
 		(tags "Cherry MX keyswitch 1.00u PCB")
@@
 	)
 	(footprint "Button_Switch_Keyboard:SW_Cherry_MX_6.25u_PCB"
+		(locked yes)
 		(layer "F.Cu")
-		(at 499.945 258.87)
+		(at 271.21 128.12)
 		(descr "Cherry MX keyswitch, 6.25u, PCB mount, http://cherryamericas.com/wp-content/uploads/2014/12/mx_cat.pdf")
 		(tags "Cherry MX keyswitch 6.25u PCB")
@@
 	)
 	(footprint "Button_Switch_Keyboard:SW_Cherry_MX_1.00u_PCB"
+		(locked yes)
 		(layer "F.Cu")
-		(at 530.44 151.76)
+		(at 358.14 108.8)
 		(descr "Cherry MX keyswitch, 1.00u, PCB mount, http://cherryamericas.com/wp-content/uploads/2014/12/mx_cat.pdf")
 		(tags "Cherry MX keyswitch 1.00u PCB")
@@
 	)
 	(footprint "Button_Switch_Keyboard:SW_Cherry_MX_1.00u_PCB"
+		(locked yes)
 		(layer "F.Cu")
-		(at 545.53 121.58)
+		(at 200.55 128.1)
 		(descr "Cherry MX keyswitch, 1.00u, PCB mount, http://cherryamericas.com/wp-content/uploads/2014/12/mx_cat.pdf")
 		(tags "Cherry MX keyswitch 1.00u PCB")
@@
 	)
 	(footprint "Button_Switch_Keyboard:SW_Cherry_MX_2.75u_PCB"
+		(locked yes)
 		(layer "F.Cu")
-		(at 567.475 162.59)
+		(at 394.84 108.72)
 		(descr "Cherry MX keyswitch, 2.75u, PCB mount, http://cherryamericas.com/wp-content/uploads/2014/12/mx_cat.pdf")
 		(tags "Cherry MX keyswitch 2.75u PCB")
@@
 	)
 	(footprint "Button_Switch_Keyboard:SW_Cherry_MX_1.00u_PCB"
+		(locked yes)
 		(layer "F.Cu")
-		(at 530.44 242.3)
+		(at 181.15 128.2)
 		(descr "Cherry MX keyswitch, 1.00u, PCB mount, http://cherryamericas.com/wp-content/uploads/2014/12/mx_cat.pdf")
 		(tags "Cherry MX keyswitch 1.00u PCB")
@@
 	)
 	(footprint "Button_Switch_Keyboard:SW_Cherry_MX_1.00u_PCB"
+		(locked yes)
 		(layer "F.Cu")
-		(at 500.26 212.12)
+		(at 220.1 108.7)
 		(descr "Cherry MX keyswitch, 1.00u, PCB mount, http://cherryamericas.com/wp-content/uploads/2014/12/mx_cat.pdf")
 		(tags "Cherry MX keyswitch 1.00u PCB")
@@
 		)
 	)
+	(group ""
+		(locked yes)
+		(members "052a2a23-c6eb-4ed9-bfd7-2b49bc2c5ffe" "1296f65c-af54-469f-8dfc-b4a44fd5d407"
+			"2894484b-00eb-4f93-a4d7-cf75be9e737c" "33b86a44-3158-4fb6-bd3c-0a80480a62ec"
+			"436b2ded-8389-42d2-9bed-1c9cae9b37fa" "52b727a2-a24a-4391-abc4-37496c2ce4d3"
+			"6a30acef-1845-4567-9fa7-2fd77dd81cdc" "a380248d-ab8f-4c0d-b550-ffea56b9dadb"
+			"a4213428-ec97-45b4-aff5-1c6b7f504b8d" "b24127f9-78a8-4276-951e-b00ce3b54ee7"
+			"c4184df0-6bbf-4e4d-b882-5865e295128e" "f7a3e06c-7f02-4e3c-b70f-b12735fa1635"
+		)
+	)
+	(group ""
+		(locked yes)
+		(members "19d5792e-d4cf-4936-9c59-56f08209b196" "283a848b-a3cb-4a78-b7c5-5718bf062408"
+			"8d47c083-7134-4056-b614-1a3adfa935cf" "8ecb330f-5e00-4146-901b-1194207d882b"
+			"9ac495a0-2730-4fea-9571-35c0e25f4158" "a8ad0a77-e800-4975-b381-176f17e219ed"
+			"a9843f3f-d519-483b-8852-6b95ed551cc6" "b33390f2-7696-46ee-ae81-893cfc0f279e"
+			"e38270c2-8ea2-44ad-a208-ed453a7c6f6a"
+		)
+	)
