File: KeebWithoutACase/KeebWithoutACase.kicad_pcb (KiCad board)
At the start: 2 copper layers, 134 parts, among them SW1 SW_Push_45deg, SW10 SW_Push_45deg, SW11 SW_Push_45deg, SW12 SW_Push_45deg, SW13 SW_Push_45deg, SW14 2U, SW15 1.5U, SW16 SW_Push_45deg, SW17 SW_Push_45deg, SW18 SW_Push_45deg, SW19 SW_Push_45deg, SW2 SW_Push_45deg, SW20 SW_Push_45deg, SW21 SW_Push_45deg, SW22 SW_Push_45deg, SW23 SW_Push_45deg, SW24 SW_Push_45deg, SW25 SW_Push_45deg, SW26 SW_Push_45deg, SW27 SW_Push_45deg, SW28 1.5U, SW29 1.75U, SW3 SW_Push_45deg, SW30 2.25U, SW31 SW_Push_45deg, SW32 SW_Push_45deg, SW33 SW_Push_45deg, SW34 SW_Push_45deg, SW35 SW_Push_45deg, SW36 SW_Push_45deg, SW37 SW_Push_45deg, SW38 SW_Push_45deg, SW39 SW_Push_45deg, SW4 SW_Push_45deg, SW40 SW_Push_45deg, SW41 SW_Push_45deg, SW42 SW_Push_45deg, SW43 SW_Push_45deg, SW44 SW_Push_45deg, SW45 SW_Push_45deg, SW46 SW_Push_45deg, SW47 SW_Push_45deg, SW48 SW_Push_45deg, SW49 SW_Push_45deg, SW5 SW_Push_45deg, SW50 SW_Push_45deg, SW51 SW_Push_45deg, SW52 2.75U, SW53 2.25U, SW54 1.25U, SW55 RotaryEncoder, SW56 SW_Push_45deg, SW57 1.25U, SW58 SW_Push_45deg, SW59 SW_Push_45deg, SW6 SW_Push_45deg, SW60 SW_Push_45deg, SW62 1.25U, SW63 SW_Push_45deg, SW64 SW_Push_45deg, SW65 SW_Push_45deg, SW66 SW_Push_45deg, SW67 SW_Push_45deg, SW7 SW_Push_45deg, SW8 SW_Push_45deg, SW9 SW_Push_45deg

Commit message: finished the media column
Parts:
- moved SW55 309.7 mm to (438.8, 56.5), turned to 180 degrees
- moved SW65 144.0 mm to (435.4, 89.2)
- moved SW66 141.0 mm to (435.4, 108.9)
- moved SW67 138.3 mm to (435.5, 128.4)
- moved SW56 138.0 mm to (435.4, 69.5)
Changed lines of the file:
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@@
 	(footprint "Button_Switch_Keyboard:SW_Cherry_MX_1.00u_PCB"
 		(layer "F.Cu")
-		(at 545.53 212.12)
+		(at 435.5 128.36)
 		(descr "Cherry MX keyswitch, 1.00u, PCB mount, http://cherryamericas.com/wp-content/uploads/2014/12/mx_cat.pdf")
 		(tags "Cherry MX keyswitch 1.00u PCB")
@@
 	(footprint "Button_Switch_Keyboard:SW_Cherry_MX_1.00u_PCB"
 		(layer "F.Cu")
-		(at 544.29 154.32)
+		(at 435.45 69.51)
 		(descr "Cherry MX keyswitch, 1.00u, PCB mount, http://cherryamericas.com/wp-content/uploads/2014/12/mx_cat.pdf")
 		(tags "Cherry MX keyswitch 1.00u PCB")
@@
 	(footprint "Rotary_Encoder:RotaryEncoder_Alps_EC11E-Switch_Vertical_H20mm"
 		(layer "F.Cu")
-		(at 741.115 -10.715)
+		(at 438.75 56.5 180)
 		(descr "Alps rotary encoder, EC11E... with switch, vertical shaft, http://www.alps.com/prod/info/E/HTML/Encoder/Incremental/EC11/EC11E15204A3.html")
 		(tags "rotary encoder")
@@
 		)
 		(property "Datasheet" "~"
-			(at 0 0 0)
+			(at 0 0 180)
 			(unlocked yes)
 			(layer "F.Fab")
@@
 		)
 		(property "Description" "Rotary encoder, dual channel, incremental quadrate outputs"
-			(at 0 0 0)
+			(at 0 0 180)
 			(unlocked yes)
 			(layer "F.Fab")
@@
 		(attr through_hole)
 		(fp_line
-			(start -0.3 -1.6)
-			(end 0.3 -1.6)
+			(start 13.6 8.4)
+			(end 9.5 8.4)
 			(stroke
 				(width 0.12)
@@
 		)
 		(fp_line
-			(start 0 -1.3)
-			(end -0.3 -1.6)
+			(start 13.6 6)
+			(end 13.6 8.4)
 			(stroke
 				(width 0.12)
@@
 		)
 		(fp_line
-			(start 0.3 -1.6)
-			(end 0 -1.3)
+			(start 13.6 1.2)
+			(end 13.6 3.8)
 			(stroke
 				(width 0.12)
@@
 		)
 		(fp_line
-			(start 1.4 -3.4)
-			(end 1.4 8.4)
+			(start 13.6 -3.4)
+			(end 13.6 -1)
 			(stroke
 				(width 0.12)
@@
 		)
 		(fp_line
-			(start 5.5 -3.4)
-			(end 1.4 -3.4)
+			(start 9.5 -3.4)
+			(end 13.6 -3.4)
 			(stroke
 				(width 0.12)
@@
 		)
 		(fp_line
-			(start 5.5 8.4)
-			(end 1.4 8.4)
+			(start 7.5 2)
+			(end 7.5 3)
 			(stroke
 				(width 0.12)
@@
 		)
 		(fp_line
-			(start 7.5 2)
-			(end 7.5 3)
+			(start 5.5 8.4)
+			(end 1.4 8.4)
 			(stroke
 				(width 0.12)
@@
 		)
 		(fp_line
-			(start 9.5 -3.4)
-			(end 13.6 -3.4)
+			(start 5.5 -3.4)
+			(end 1.4 -3.4)
 			(stroke
 				(width 0.12)
@@
 		)
 		(fp_line
-			(start 13.6 -3.4)
-			(end 13.6 -1)
+			(start 1.4 -3.4)
+			(end 1.4 8.4)
 			(stroke
 				(width 0.12)
@@
 		)
 		(fp_line
-			(start 13.6 1.2)
-			(end 13.6 3.8)
+			(start 0.3 -1.6)
+			(end 0 -1.3)
 			(stroke
 				(width 0.12)
@@
 		)
 		(fp_line
-			(start 13.6 6)
-			(end 13.6 8.4)
+			(start 0 -1.3)
+			(end -0.3 -1.6)
 			(stroke
 				(width 0.12)
@@
 		)
 		(fp_line
-			(start 13.6 8.4)
-			(end 9.5 8.4)
+			(start -0.3 -1.6)
+			(end 0.3 -1.6)
 			(stroke
 				(width 0.12)
@@
 		)
 		(fp_line
-			(start -1.5 -4.6)
-			(end -1.5 9.6)
+			(start 16 9.6)
+			(end 16 -4.6)
 			(stroke
 				(width 0.05)
@@
 		)
 		(fp_line
-			(start -1.5 -4.6)
-			(end 16 -4.6)
+			(start 16 9.6)
+			(end -1.5 9.6)
 			(stroke
 				(width 0.05)
@@
 		)
 		(fp_line
-			(start 16 9.6)
-			(end -1.5 9.6)
+			(start -1.5 -4.6)
+			(end 16 -4.6)
 			(stroke
 				(width 0.05)
@@
 		)
 		(fp_line
-			(start 16 9.6)
-			(end 16 -4.6)
+			(start -1.5 -4.6)
+			(end -1.5 9.6)
 			(stroke
 				(width 0.05)
@@
 		)
 		(fp_line
-			(start 1.5 -2.2)
-			(end 2.5 -3.3)
+			(start 13.5 8.3)
+			(end 1.5 8.3)
 			(stroke
 				(width 0.12)
@@
 		)
 		(fp_line
-			(start 1.5 8.3)
-			(end 1.5 -2.2)
+			(start 13.5 -3.3)
+			(end 13.5 8.3)
 			(stroke
 				(width 0.12)
@@
 		)
 		(fp_line
-			(start 2.5 -3.3)
-			(end 13.5 -3.3)
+			(start 7.5 -0.5)
+			(end 7.5 5.5)
 			(stroke
 				(width 0.12)
@@
 		)
 		(fp_line
-			(start 7.5 -0.5)
-			(end 7.5 5.5)
+			(start 2.5 -3.3)
+			(end 13.5 -3.3)
 			(stroke
 				(width 0.12)
@@
 		)
 		(fp_line
-			(start 13.5 -3.3)
-			(end 13.5 8.3)
+			(start 1.5 8.3)
+			(end 1.5 -2.2)
 			(stroke
 				(width 0.12)
@@
 		)
 		(fp_line
-			(start 13.5 8.3)
-			(end 1.5 8.3)
+			(start 1.5 -2.2)
+			(end 2.5 -3.3)
 			(stroke
 				(width 0.12)
@@
 		)
 		(pad "A" thru_hole rect
-			(at 0 0)
+			(at 0 0 180)
 			(size 2 2)
 			(drill 1)
@@
 		)
 		(pad "B" thru_hole circle
-			(at 0 5)
+			(at 0 5 180)
 			(size 2 2)
 			(drill 1)
@@
 		)
 		(pad "C" thru_hole circle
-			(at 0 2.5)
+			(at 0 2.5 180)
 			(size 2 2)
 			(drill 1)
@@
 		)
 		(pad "MP" thru_hole rect
-			(at 7.5 -3.1)
+			(at 7.5 -3.1 180)
 			(size 3.2 2)
 			(drill oval 2.8 1.5)
@@
 		)
 		(pad "MP" thru_hole rect
-			(at 7.5 8.1)
+			(at 7.5 8.1 180)
 			(size 3.2 2)
 			(drill oval 2.8 1.5)
@@
 		)
 		(pad "S1" thru_hole circle
-			(at 14.5 5)
+			(at 14.5 5 180)
 			(size 2 2)
 			(drill 1)
@@
 		)
 		(pad "S2" thru_hole circle
-			(at 14.5 0)
+			(at 14.5 0 180)
 			(size 2 2)
 			(drill 1)
@@
 	(footprint "Button_Switch_Keyboard:SW_Cherry_MX_1.00u_PCB"
 		(layer "F.Cu")
-		(at 545.53 197.03)
+		(at 435.45 108.86)
 		(descr "Cherry MX keyswitch, 1.00u, PCB mount, http://cherryamericas.com/wp-content/uploads/2014/12/mx_cat.pdf")
 		(tags "Cherry MX keyswitch 1.00u PCB")
@@
 	(footprint "Button_Switch_Keyboard:SW_Cherry_MX_1.00u_PCB"
 		(layer "F.Cu")
-		(at 545.53 181.94)
+		(at 435.45 89.16)
 		(descr "Cherry MX keyswitch, 1.00u, PCB mount, http://cherryamericas.com/wp-content/uploads/2014/12/mx_cat.pdf")
 		(tags "Cherry MX keyswitch 1.00u PCB")
@@
 		)
 	)
+	(group ""
+		(members "2583b367-aeb6-44ad-816a-34be03c0951b" "519b5d4d-062b-48f7-b44c-a297db88cfc3"
+			"807238b1-67d4-4dde-a6d1-12be65fd5f5c" "939f7f53-c0a8-465e-88a2-a185328ba31e"
+			"e3ec9077-a84d-481d-9317-26dd73b0cbb0"
+		)
+	)

Commit message: added the diodes for the first row
Parts:
- D1: moved to B.Cu
- moved D1 571.1 mm to (142.8, 61.0), turned to 180 degrees
- moved D2 550.4 mm to (162.4, 61.0), turned to 180 degrees
- moved D3 529.9 mm to (181.7, 61.0), turned to 180 degrees
- moved D4 509.2 mm to (201.2, 61.0), turned to 180 degrees
- moved D5 488.4 mm to (220.8, 60.9), turned to 180 degrees
- moved D6 467.6 mm to (240.5, 60.8), turned to 180 degrees
- moved D7 446.7 mm to (260.1, 60.5), turned to 180 degrees
- moved D8 426.0 mm to (279.8, 60.6), turned to 180 degrees
- moved D9 405.1 mm to (299.5, 60.5), turned to 180 degrees
- moved D10 384.3 mm to (319.1, 60.5), turned to 180 degrees
- moved D11 363.6 mm to (338.6, 60.5), turned to 180 degrees
- moved D12 342.8 mm to (358.4, 60.5), turned to 180 degrees
- moved D13 322.2 mm to (377.8, 60.5), turned to 180 degrees
- moved D14 292.2 mm to (407.1, 60.8), turned to 180 degrees
- moved D58 176.4 mm to (703.4, 56.5), turned to 180 degrees
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
Commit message: added all the diodes fr the 2nd row
Parts:
- moved D15 614.0 mm to (147.4, 80.5)
- moved D16 590.1 mm to (171.7, 80.5)
- moved D17 570.9 mm to (191.3, 80.4)
- moved D18 551.7 mm to (211.1, 80.3)
- moved D19 533.0 mm to (230.4, 80.2)
- moved D20 514.2 mm to (250.1, 80.2)
- moved D21 495.5 mm to (269.7, 80.1)
- moved D22 477.1 mm to (289.4, 80.2)
- moved D23 458.6 mm to (309.2, 80.2)
- moved D24 440.6 mm to (328.8, 80.2)
- moved D25 422.7 mm to (348.5, 80.2)
- moved D26 405.3 mm to (368.0, 79.9)
- moved D27 388.0 mm to (387.7, 79.8)
- moved D28 367.1 mm to (411.6, 79.8)
- moved A1 338.0 mm to (537.0, 184.6)
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