File: KeebWithoutACase/KeebWithoutACase.kicad_pcb (KiCad board)
At the start: 2 copper layers, 134 parts, among them SW1 SW_Push_45deg, SW10 SW_Push_45deg, SW11 SW_Push_45deg, SW12 SW_Push_45deg, SW13 SW_Push_45deg, SW14 2U, SW15 1.5U, SW16 SW_Push_45deg, SW17 SW_Push_45deg, SW18 SW_Push_45deg, SW19 SW_Push_45deg, SW2 SW_Push_45deg, SW20 SW_Push_45deg, SW21 SW_Push_45deg, SW22 SW_Push_45deg, SW23 SW_Push_45deg, SW24 SW_Push_45deg, SW25 SW_Push_45deg, SW26 SW_Push_45deg, SW27 SW_Push_45deg, SW28 1.5U, SW29 1.75U, SW3 SW_Push_45deg, SW30 2.25U, SW31 SW_Push_45deg, SW32 SW_Push_45deg, SW33 SW_Push_45deg, SW34 SW_Push_45deg, SW35 SW_Push_45deg, SW36 SW_Push_45deg, SW37 SW_Push_45deg, SW38 SW_Push_45deg, SW39 SW_Push_45deg, SW4 SW_Push_45deg, SW40 SW_Push_45deg, SW41 SW_Push_45deg, SW42 SW_Push_45deg, SW43 SW_Push_45deg, SW44 SW_Push_45deg, SW45 SW_Push_45deg, SW46 SW_Push_45deg, SW47 SW_Push_45deg, SW48 SW_Push_45deg, SW49 SW_Push_45deg, SW5 SW_Push_45deg, SW50 SW_Push_45deg, SW51 SW_Push_45deg, SW52 2.75U, SW53 2.25U, SW54 1.25U, SW55 RotaryEncoder, SW56 SW_Push_45deg, SW57 1.25U, SW58 SW_Push_45deg, SW59 SW_Push_45deg, SW6 SW_Push_45deg, SW60 SW_Push_45deg, SW62 1.25U, SW63 SW_Push_45deg, SW64 SW_Push_45deg, SW65 SW_Push_45deg, SW66 SW_Push_45deg, SW67 SW_Push_45deg, SW7 SW_Push_45deg, SW8 SW_Push_45deg, SW9 SW_Push_45deg

Commit message: placed rest of the diodes
Parts:
- moved D29 448.7 mm to (149.8, 100.0)
- moved D30 431.9 mm to (154.4, 119.5)
- moved D31 418.5 mm to (176.4, 100.5)
- moved D32 397.5 mm to (185.8, 119.8)
- moved D33 394.8 mm to (195.8, 100.3)
- moved D57 386.2 mm to (144.7, 138.9)
- moved D58 381.0 mm to (166.9, 139.2)
- moved D34 373.7 mm to (205.6, 119.8)
- moved D35 371.1 mm to (215.3, 100.3)
- moved D59 360.7 mm to (186.3, 139.3)
- moved D36 349.9 mm to (225.2, 119.8)
- moved D37 347.3 mm to (234.9, 100.2)
- moved D60 341.1 mm to (205.3, 138.7)
- moved D38 325.9 mm to (245.1, 120.0)
- moved D39 323.4 mm to (254.6, 100.2)
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