File: KeebWithoutACase/KeebWithoutACase.kicad_pcb (KiCad board)
At the start: 2 copper layers, 134 parts, among them SW1 SW_Push_45deg, SW10 SW_Push_45deg, SW11 SW_Push_45deg, SW12 SW_Push_45deg, SW13 SW_Push_45deg, SW14 2U, SW15 1.5U, SW16 SW_Push_45deg, SW17 SW_Push_45deg, SW18 SW_Push_45deg, SW19 SW_Push_45deg, SW2 SW_Push_45deg, SW20 SW_Push_45deg, SW21 SW_Push_45deg, SW22 SW_Push_45deg, SW23 SW_Push_45deg, SW24 SW_Push_45deg, SW25 SW_Push_45deg, SW26 SW_Push_45deg, SW27 SW_Push_45deg, SW28 1.5U, SW29 1.75U, SW3 SW_Push_45deg, SW30 2.25U, SW31 SW_Push_45deg, SW32 SW_Push_45deg, SW33 SW_Push_45deg, SW34 SW_Push_45deg, SW35 SW_Push_45deg, SW36 SW_Push_45deg, SW37 SW_Push_45deg, SW38 SW_Push_45deg, SW39 SW_Push_45deg, SW4 SW_Push_45deg, SW40 SW_Push_45deg, SW41 SW_Push_45deg, SW42 SW_Push_45deg, SW43 SW_Push_45deg, SW44 SW_Push_45deg, SW45 SW_Push_45deg, SW46 SW_Push_45deg, SW47 SW_Push_45deg, SW48 SW_Push_45deg, SW49 SW_Push_45deg, SW5 SW_Push_45deg, SW50 SW_Push_45deg, SW51 SW_Push_45deg, SW52 2.75U, SW53 2.25U, SW54 1.25U, SW55 RotaryEncoder, SW56 SW_Push_45deg, SW57 1.25U, SW58 SW_Push_45deg, SW59 SW_Push_45deg, SW6 SW_Push_45deg, SW60 SW_Push_45deg, SW62 1.25U, SW63 SW_Push_45deg, SW64 SW_Push_45deg, SW65 SW_Push_45deg, SW66 SW_Push_45deg, SW67 SW_Push_45deg, SW7 SW_Push_45deg, SW8 SW_Push_45deg, SW9 SW_Push_45deg

Commit message: wired the switches with their respective diodes
Routing:
- net Net-(D31-A): track 0.00 -> 10.4 mm
- net Net-(D33-A): track 0.00 -> 10.3 mm
- net Net-(D38-A): track 0.00 -> 10.3 mm
- net Net-(D35-A): track 0.00 -> 10.3 mm
- net Net-(D3-A): track 0.00 -> 10.2 mm
- net Net-(D39-A): track 0.00 -> 10.2 mm
- net Net-(D59-A): track 0.00 -> 10.2 mm
- net Net-(D37-A): track 0.00 -> 10.2 mm
- net Net-(D45-A): track 0.00 -> 10.2 mm
- net Net-(D4-A): track 0.00 -> 10.1 mm
- net Net-(D34-A): track 0.00 -> 10.1 mm
- net Net-(D32-A): track 0.00 -> 10.1 mm
- net Net-(D41-A): track 0.00 -> 10.1 mm
- net Net-(D17-A): track 0.00 -> 10.1 mm
- net Net-(D36-A): track 0.00 -> 10.1 mm
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
Commit message: fixed the schm col1 bleeding
Routing:
- net COL 1: track 0.00 -> 648.5 mm
- net ROW 2: track 0.00 -> 338.5 mm
- net ROW 3: track 0.00 -> 334.7 mm
- net ROW 1: track 0.00 -> 304.8 mm

Commit message: fixed wiring the switch matrix
Connections:
- A1 pad 10: COL 1 -> COL 3
- A1 pad 11: COL 1 -> COL 4
- A1 pad 12: COL 1 -> COL 5
- A1 pad 14: COL 1 -> COL 6
- A1 pad 15: COL 1 -> COL 7
- A1 pad 16: COL 1 -> COL 8
- A1 pad 17: COL 1 -> COL 9
- A1 pad 19: COL 1 -> COL 10
- A1 pad 20: COL 1 -> COL 11
- A1 pad 21: COL 1 -> COL 12
- A1 pad 25: COL 1 -> COL 15
- A1 pad 5: COL 1 -> ROW 4
- A1 pad 6: COL 1 -> ROW 5
- D30 pad 1: COL 1 -> ROW 4
- D32 pad 1: COL 1 -> ROW 4
- D34 pad 1: COL 1 -> ROW 4
- D36 pad 1: COL 1 -> ROW 4
- D38 pad 1: COL 1 -> ROW 4
- D40 pad 1: COL 1 -> ROW 4
- D42 pad 1: COL 1 -> ROW 4
- D44 pad 1: COL 1 -> ROW 4
- D46 pad 1: COL 1 -> ROW 4
- D48 pad 1: COL 1 -> ROW 4
- D50 pad 1: COL 1 -> ROW 4
- D52 pad 1: COL 1 -> ROW 4
- D54 pad 1: COL 1 -> ROW 5
- D57 pad 1: COL 1 -> ROW 5
- D58 pad 1: COL 1 -> ROW 5
- D59 pad 1: COL 1 -> ROW 5
- D60 pad 1: COL 1 -> ROW 5
- D61 pad 1: COL 1 -> ROW 5
- D62 pad 1: COL 1 -> ROW 5
- D63 pad 1: COL 1 -> ROW 5
- D64 pad 1: COL 1 -> ROW 5
- D66 pad 1: COL 1 -> ROW 4
- D67 pad 1: COL 1 -> ROW 5
- SW10 pad 1: COL 1 -> COL 10
- SW11 pad 1: COL 1 -> COL 11
- SW12 pad 1: COL 1 -> COL 12
- SW16 pad 1: COL 1 -> COL2
- SW17 pad 1: COL 1 -> COL 3
- SW18 pad 1: COL 1 -> COL 4
- SW19 pad 1: COL 1 -> COL 5
- SW2 pad 1: COL 1 -> COL2
- SW20 pad 1: COL 1 -> COL 6
- SW21 pad 1: COL 1 -> COL 7
- SW22 pad 1: COL 1 -> COL 8
- SW23 pad 1: COL 1 -> COL 9
- SW24 pad 1: COL 1 -> COL 10
- SW25 pad 1: COL 1 -> COL 11
- SW26 pad 1: COL 1 -> COL 12
- SW3 pad 1: COL 1 -> COL 3
- SW31 pad 1: COL 1 -> COL2
- SW32 pad 1: COL 1 -> COL2
- SW33 pad 1: COL 1 -> COL 3
- SW34 pad 1: COL 1 -> COL 3
- SW35 pad 1: COL 1 -> COL 4
- SW36 pad 1: COL 1 -> COL 4
- SW37 pad 1: COL 1 -> COL 5
- SW38 pad 1: COL 1 -> COL 5
- SW39 pad 1: COL 1 -> COL 6
- SW4 pad 1: COL 1 -> COL 4
- SW40 pad 1: COL 1 -> COL 6
- SW41 pad 1: COL 1 -> COL 7
- SW42 pad 1: COL 1 -> COL 7
- SW43 pad 1: COL 1 -> COL 8
- SW44 pad 1: COL 1 -> COL 8
- SW45 pad 1: COL 1 -> COL 9
- SW46 pad 1: COL 1 -> COL 9
- SW47 pad 1: COL 1 -> COL 10
- SW48 pad 1: COL 1 -> COL 10
- SW49 pad 1: COL 1 -> COL 11
- SW5 pad 1: COL 1 -> COL 5
- SW50 pad 1: COL 1 -> COL 11
- SW51 pad 1: COL 1 -> COL 12
- SW52 pad 1: COL 1 -> COL 12
- SW56 pad 1: COL 1 -> COL 15
- SW58 pad 1: COL 1 -> COL2
- SW59 pad 1: COL 1 -> COL 3
- SW6 pad 1: COL 1 -> COL 6
- SW60 pad 1: COL 1 -> COL 4
- SW62 pad 1: COL 1 -> COL 6
- SW63 pad 1: COL 1 -> COL 7
- SW64 pad 1: COL 1 -> COL 8
- SW65 pad 1: COL 1 -> COL 15
- SW66 pad 1: COL 1 -> COL 15
- SW67 pad 1: unconnected-(SW67-Pad1) -> COL 15
- SW7 pad 1: COL 1 -> COL 7
- SW8 pad 1: COL 1 -> COL 8
- SW9 pad 1: COL 1 -> COL 9
- SpaceBar1 pad 1: COL 1 -> COL 5
Routing:
- net COL 1: track 648.5 -> 87.1 mm
- net ROW 4: track 0.00 -> 340.6 mm
- net ROW 5: track 0.00 -> 307.9 mm
- net COL 5: track 0.00 -> 108.2 mm
- net COL 3: track 0.00 -> 97.2 mm
- net COL 4: track 0.00 -> 96.9 mm
- net COL2: track 0.00 -> 96.7 mm
- net COL 12: track 0.00 -> 80.2 mm
- net COL 11: track 0.00 -> 69.2 mm
- net COL 9: track 0.00 -> 69.1 mm
- net COL 10: track 0.00 -> 69.1 mm
- net COL 7: track 0.00 -> 69.1 mm
- net COL 8: track 0.00 -> 69.1 mm
- net COL 6: track 0.00 -> 68.9 mm
- net COL 15: track 0.00 -> 58.9 mm
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
Commit message: wired all the stuff to the mcu and completed the wiring of the pcb for the keyboard
Parts:
- moved A1 441.5 mm to (111.2, 68.0), turned to 0 degrees
Connections:
- A1 pad 13: Net-(A1-GND-Pad13) -> GND
- A1 pad 18: Net-(A1-GND-Pad13) -> GND
- A1 pad 23: Net-(A1-GND-Pad13) -> GND
- A1 pad 27: ENCODER B -> unconnected-(A1-GPIO21-Pad27)
- A1 pad 28: Net-(A1-GND-Pad13) -> GND
- A1 pad 3: Net-(A1-GND-Pad13) -> GND
- A1 pad 38: Net-(A1-GND-Pad13) -> GND
- A1 pad 8: Net-(A1-GND-Pad13) -> GND
- SW16 pad 1: COL2 -> COL 2
- SW2 pad 1: COL2 -> COL 2
- SW31 pad 1: COL2 -> COL 2
- SW32 pad 1: COL2 -> COL 2
- SW58 pad 1: COL2 -> COL 2
Routing:
- net COL 8: track 69.1 -> 704.6 mm
- net ENCODER A: track 0.00 -> 511.5 mm, vias 0 -> 2
- net GND: track 0.00 -> 504.8 mm
- net COL 14: track 21.4 -> 490.0 mm, vias 0 -> 2
- net COL 12: track 80.2 -> 461.4 mm, vias 0 -> 1
- net COL 5: track 108.2 -> 482.7 mm, vias 0 -> 2
- net COL 15: track 58.9 -> 431.4 mm, vias 0 -> 3
- net ENCODER B: track 0.00 -> 329.2 mm, vias 0 -> 1
- net COL 13: track 54.8 -> 369.0 mm, vias 0 -> 2
- net COL 7: track 69.1 -> 367.6 mm, vias 0 -> 3
- net COL 11: track 69.2 -> 363.9 mm
- net COL 6: track 68.9 -> 343.0 mm, vias 0 -> 4
- net COL 10: track 69.1 -> 340.7 mm
- net COL 9: track 69.1 -> 314.6 mm
- net COL 2: track 0.00 -> 164.0 mm
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
Commit message: wired the pcb cut the edges added serations ettc etc
Parts:
- added REF**: MountingHole_2.1mm, MountingHole:MountingHole_2.1mm, F.Cu at (193.5, 32.5)
- added REF**: MountingHole_2.1mm, MountingHole:MountingHole_2.1mm, F.Cu at (356.0, 32.5)
- added REF**: MountingHole_2.1mm, MountingHole:MountingHole_2.1mm, F.Cu at (88.5, 83.5)
- added REF**: MountingHole_2.1mm, MountingHole:MountingHole_2.1mm, F.Cu at (99.5, 121.5)
- added REF**: MountingHole_2.1mm, MountingHole:MountingHole_2.1mm, F.Cu at (452.5, 92.5)
- added REF**: MountingHole_2.1mm, MountingHole:MountingHole_2.1mm, F.Cu at (450.5, 33.5)
- added REF**: MountingHole_2.1mm, MountingHole:MountingHole_2.1mm, F.Cu at (121.5, 151.5)
- added REF**: PinHeader_1x02_P1.00mm_Vertical, Connector_PinHeader_1.00mm:PinHeader_1x02_P1.00mm_Vertical, F.Cu at (440.5, 42.5)
- added REF**: MountingHole_2.1mm, MountingHole:MountingHole_2.1mm, F.Cu at (449.0, 148.0)
- added REF**: MountingHole_2.1mm, MountingHole:MountingHole_2.1mm, F.Cu at (87.5, 32.5)
- added REF**: MountingHole_2.1mm, MountingHole:MountingHole_2.1mm, F.Cu at (277.5, 33.0)
Routing:
- net COL 13: track 369.0 -> 384.2 mm
- net COL 5: track 482.7 -> 489.0 mm
- net COL 3: track 221.1 -> 227.4 mm
- net COL 2: track 164.0 -> 169.6 mm
- net ROW 2: track 376.4 -> 381.3 mm
- net ROW 4: track 412.4 -> 416.4 mm
- net GND: track 504.8 -> 508.5 mm
- net COL 14: track 490.0 -> 493.6 mm
- net ROW 1: track 329.4 -> 332.8 mm
- net ROW 3: track 388.0 -> 390.7 mm
- net ENCODER A: track 511.5 -> 513.4 mm
- net COL 15: track 431.4 -> 432.6 mm
Other:
- board outline added: 373.5 x 126.5 mm
